File: macroKeyPad.kicad_pcb (KiCad board)
At the start: 2 copper layers, 102.3 x 39.6 mm, 19 parts, among them U1 kb2040

Commit message: finalizing art and creating housing
Parts:
- moved G*** 12.1 mm to (65.5, 67.3)

Commit message: added final touches
gonna have it checked and then purchase the board
Routing:
- added copper zone on B.Cu, net (none)
- added copper zone on F.Cu, net (none)

Commit message: ordered!
Routing:
- net Row0: track 86.5 -> 83.0 mm
- net Row1: track 82.1 -> 78.9 mm
Changed lines of the file:
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@@
 			(layer "F.Mask")
 		)
-		(fp_poly
-			(pts
-				(xy -0.121616 -12.596959) (xy -0.030644 -12.590156) (xy -0.012483 -12.580646) (xy -0.059445 -12.540167)
-				(xy -0.159694 -12.455954) (xy -0.296653 -12.341885) (xy -0.398728 -12.257295) (xy -0.572001 -12.118296)
-				(xy -0.701528 -12.028398) (xy -0.810041 -11.975218) (xy -0.920275 -11.946373) (xy -0.98732 -11.936701)
-				(xy -1.108672 -11.926534) (xy -1.27531 -11.91835) (xy -1.46797 -11.912369) (xy -1.667387 -11.908807)
-				(xy -1.854296 -11.907882) (xy -2.009432 -11.909813) (xy -2.113529 -11.914816) (xy -2.147323 -11.923111)
-				(xy -2.146851 -11.923591) (xy -2.102403 -11.949631) (xy -1.992713 -12.010628) (xy -1.832271 -12.098612)
-				(xy -1.635568 -12.205613) (xy -1.539395 -12.257676) (xy -0.950803 -12.575836) (xy -0.465246 -12.593743)
-				(xy -0.272099 -12.598317)
-			)
-			(stroke
-				(width 0)
-				(type solid)
-			)
-			(fill yes)
-			(layer "F.Paste")
-		)
-		(fp_poly
-			(pts
-				(xy 3.072403 -24.145066) (xy 3.529182 -24.127707) (xy 3.937197 -24.099454) (xy 4.210695 -24.069329)
-				(xy 5.315958 -23.878843) (xy 6.374384 -23.612865) (xy 7.392282 -23.269219) (xy 8.375967 -22.845727)
-				(xy 9.331748 -22.340212) (xy 9.486668 -22.249089) (xy 9.785967 -22.062662) (xy 10.111445 -21.846495)
-				(xy 10.444366 -21.614141) (xy 10.765994 -21.379153) (xy 11.057594 -21.155085) (xy 11.300429 -20.955489)
-				(xy 11.409625 -20.858068) (xy 11.636007 -20.647281) (xy 11.235507 -20.829363) (xy 10.365656 -21.175183)
-				(xy 9.459396 -21.438612) (xy 8.518836 -21.61921) (xy 7.546082 -21.716538) (xy 6.88773 -21.734947)
-				(xy 6.232068 -21.720122) (xy 5.628997 -21.672646) (xy 5.045192 -21.588479) (xy 4.447331 -21.463584)
-				(xy 4.252655 -21.415641) (xy 3.312279 -21.130485) (xy 2.408845 -20.763184) (xy 1.5459 -20.315619)
-				(xy 0.726992 -19.789668) (xy -0.044331 -19.187211) (xy -0.182813 -19.066379) (xy -0.327646 -18.944121)
-				(xy -0.453498 -18.849293) (xy -0.541301 -18.795772) (xy -0.564206 -18.788829) (xy -0.633767 -18.775269)
-				(xy -0.768698 -18.739166) (xy -0.948366 -18.686309) (xy -1.11707 -18.633736) (xy -1.352959 -18.548862)
-				(xy -1.591424 -18.441821) (xy -1.844497 -18.305454) (xy -2.124211 -18.132604) (xy -2.442597 -17.916112)
-				(xy -2.811689 -17.648821) (xy -2.965598 -17.534051) (xy -3.203688 -17.345733) (xy -3.480142 -17.110876)
-				(xy -3.785362 -16.838987) (xy -4.109748 -16.539574) (xy -4.443703 -16.222145) (xy -4.777627 -15.896208)
-				(xy -5.101921 -15.571271) (xy -5.406986 -15.256841) (xy -5.683224 -14.962427) (xy -5.921036 -14.697535)
-				(xy -6.110822 -14.471674) (xy -6.242985 -14.294352) (xy -6.255327 -14.275527) (xy -6.406596 -14.040001)
-				(xy -6.406596 -13.432289) (xy -6.400199 -13.090667) (xy -6.381127 -12.833909) (xy -6.349562 -12.664274)
-				(xy -6.34387 -12.646791) (xy -6.303994 -12.520561) (xy -6.252305 -12.338869) (xy -6.197968 -12.134339)
-				(xy -6.180127 -12.063826) (xy -6.112974 -11.811602) (xy -6.049883 -11.624223) (xy -5.979437 -11.477312)
-				(xy -5.890215 -11.346496) (xy -5.787536 -11.225817) (xy -5.689113 -11.124261) (xy -5.605764 -11.071005)
-				(xy -5.500677 -11.050563) (xy -5.363501 -11.047416) (xy -5.211161 -11.051522) (xy -5.112876 -11.07472)
-				(xy -5.032189 -11.133333) (xy -4.937304 -11.238237) (xy -4.830391 -11.392128) (xy -4.731284 -11.582345)
-				(xy -4.683992 -11.702319) (xy -4.594014 -11.97558) (xy -4.620754 -11.61337) (xy -4.642391 -11.42048)
-				(xy -4.680679 -11.173602) (xy -4.729934 -10.906499) (xy -4.776996 -10.685206) (xy -4.828795 -10.472618)
-				(xy -4.884659 -10.277957) (xy -4.951665 -10.082493) (xy -5.036885 -9.867497) (xy -5.147397 -9.614238)
-				(xy -5.290273 -9.303987) (xy -5.333634 -9.211593) (xy -5.462352 -8.930315) (xy -5.602152 -8.611427)
-				(xy -5.747387 -8.269097) (xy -5.892408 -7.917493) (xy -6.03157 -7.570781) (xy -6.159224 -7.243131)
-				(xy -6.269724 -6.948709) (xy -6.357422 -6.701683) (xy -6.416671 -6.516221) (xy -6.433662 -6.451872)
-				(xy -6.46675 -6.355256) (xy -6.53121 -6.2019) (xy -6.616734 -6.015459) (xy -6.684863 -5.875422)
-				(xy -6.775767 -5.68189) (xy -6.848351 -5.505896) (xy -6.893751 -5.37026) (xy -6.904635 -5.309609)
-				(xy -6.923842 -5.231046) (xy -6.977345 -5.086265) (xy -7.058969 -4.890051) (xy -7.162539 -4.657193)
-				(xy -7.281878 -4.402475) (xy -7.294098 -4.377083) (xy -7.438301 -4.073639) (xy -7.545398 -3.836208)
-				(xy -7.62077 -3.650834) (xy -7.669797 -3.503564) (xy -7.697859 -3.380442) (xy -7.707599 -3.304657)
-				(xy -7.722493 -3.170648) (xy -7.748167 -3.076874) (xy -7.800335 -2.998009) (xy -7.894707 -2.908727)
-				(xy -8.014386 -2.810157) (xy -8.149014 -2.70329) (xy -8.255753 -2.622964) (xy -8.316201 -2.58289)
-				(xy -8.322266 -2.58075) (xy -8.354407 -2.616541) (xy -8.427349 -2.715578) (xy -8.532286 -2.865352)
-				(xy -8.660408 -3.053354) (xy -8.760695 -3.203299) (xy -9.017844 -3.614073) (xy -9.285084 -4.082844)
-				(xy -9.54914 -4.583522) (xy -9.796736 -5.090017) (xy -10.014598 -5.57624) (xy -10.183224 -5.99911)
-				(xy -10.455229 -6.832083) (xy -10.68147 -7.722736) (xy -10.85651 -8.647671) (xy -10.940586 -9.259003)
-				(xy -10.966069 -9.555771) (xy -10.982906 -9.920226) (xy -10.991283 -10.329934) (xy -10.991383 -10.762463)
-				(xy -10.983393 -11.195377) (xy -10.967495 -11.606243) (xy -10.943876 -11.972627) (xy -10.915985 -12.247238)
-				(xy -10.7664 -13.196726) (xy -10.565168 -14.090826) (xy -10.30527 -14.95294) (xy -9.979689 -15.806469)
-				(xy -9.599054 -16.639038) (xy -9.093465 -17.572888) (xy -8.519925 -18.453851) (xy -7.87257 -19.29008)
-				(xy -7.145537 -20.089729) (xy -7.041762 -20.194525) (xy -6.219948 -20.954536) (xy -5.353456 -21.635837)
-				(xy -4.442931 -22.238111) (xy -3.489014 -22.761044) (xy -2.492347 -23.204322) (xy -1.453574 -23.567628)
-				(xy -0.373337 -23.850648) (xy 0.747721 -24.053067) (xy 0.860249 -24.068622) (xy 1.216622 -24.105659)
-				(xy 1.638971 -24.131828) (xy 2.10435 -24.147121) (xy 2.58981 -24.151536)
-			)
-			(stroke
-				(width 0)
-				(type solid)
-			)
-			(fill yes)
-			(layer "F.Paste")
-		)
 		(embedded_fonts no)
 	)
@@
 			(at 0 0 0)
 			(layer "F.SilkS")
+			(hide yes)
 			(effects
 				(font
@@
 	)
 	(segment
-		(start 100.1875 48)
-		(end 101.9875 46.2)
+		(start 100.15 47.93)
+		(end 98.42 46.2)
 		(width 0.2)
 		(layer "F.Cu")
@@
 	)
 	(segment
-		(start 137.3875 48)
-		(end 139.1875 46.2)
+		(start 135.55 46.2)
+		(end 137.35 48)
 		(width 0.2)
 		(layer "F.Cu")
@@
 	)
 	(segment
-		(start 156 47.9875)
-		(end 157.7875 46.2)
+		(start 154.3 46.2)
+		(end 154.3 46.3)
 		(width 0.2)
 		(layer "F.Cu")
@@
 	)
 	(segment
-		(start 118.7875 48)
-		(end 120.5875 46.2)
+		(start 100.15 48)
+		(end 100.15 47.93)
+		(width 0.2)
+		(layer "F.Cu")
+		(net 1)
+	)
+	(segment
+		(start 116.95 46.2)
+		(end 118.75 48)
+		(width 0.2)
+		(layer "F.Cu")
+		(net 1)
+	)
+	(segment
+		(start 154.3 46.3)
+		(end 156 48)
 		(width 0.2)
 		(layer "F.Cu")
@@
 	)
 	(via
-		(at 101.9875 46.2)
+		(at 98.42 46.2)
 		(size 0.7)
 		(drill 0.4)
@@
 	)
 	(via
-		(at 157.7875 46.2)
+		(at 135.55 46.2)
 		(size 0.7)
 		(drill 0.4)
@@
 	)
 	(via
-		(at 139.1875 46.2)
+		(at 154.3 46.2)
 		(size 0.7)
 		(drill 0.4)
@@
 	)
 	(via
-		(at 120.5875 46.2)
+		(at 116.95 46.2)
 		(size 0.7)
 		(drill 0.4)
@@
 	(segment
 		(start 97.760108 46.2)
-		(end 101.9875 46.2)
+		(end 99.69 46.2)
 		(width 0.2)
 		(layer "B.Cu")
@@
 	)
 	(segment
-		(start 101.9875 46.2)
+		(start 117.47 46.2)
 		(end 120.5875 46.2)
 		(width 0.2)
@@
 	)
 	(segment
+		(start 101.9875 46.2)
+		(end 117.47 46.2)
+		(width 0.2)
+		(layer "B.Cu")
+		(net 1)
+	)
+	(segment
 		(start 139.1875 46.2)
-		(end 120.5875 46.2)
+		(end 136.52 46.2)
+		(width 0.2)
+		(layer "B.Cu")
+		(net 1)
+	)
+	(segment
+		(start 154.3 46.2)
+		(end 139.1875 46.2)
+		(width 0.2)
+		(layer "B.Cu")
+		(net 1)
+	)
+	(segment
+		(start 99.69 46.2)
+		(end 101.9875 46.2)
 		(width 0.2)
 		(layer "B.Cu")
@@
 	)
 	(segment
-		(start 157.7875 46.2)
-		(end 139.1875 46.2)
+		(start 136.52 46.2)
+		(end 120.5875 46.2)
 		(width 0.2)
 		(layer "B.Cu")
@@
 	)
 	(segment
+		(start 100.15 65.5)
+		(end 98.5 63.85)
+		(width 0.2)
+		(layer "F.Cu")
+		(net 7)
+	)
+	(segment
 		(start 120.5875 63.8)
-		(end 139.1875 63.8)
+		(end 135.25 63.8)
 		(width 0.2)
 		(layer "F.Cu")
@@
 	)
 	(segment
-		(start 137.3 65.5)
-		(end 137.4875 65.5)
+		(start 155.9 65.5)
+		(end 154.3 63.9)
 		(width 0.2)
 		(layer "F.Cu")
@@
 	)
 	(segment
-		(start 118.8875 65.5)
-		(end 120.5875 63.8)
+		(start 137.3 65.5)
+		(end 137.4875 65.5)
 		(width 0.2)
 		(layer "F.Cu")
@@
 	)
 	(segment
+		(start 154.3 63.9)
+		(end 154.3 63.8)
+		(width 0.2)
+		(layer "F.Cu")
+		(net 7)
+	)
+	(segment
+		(start 137.3 65.5)
+		(end 135.6 63.8)
+		(width 0.2)
+		(layer "F.Cu")
+		(net 7)
+	)
+	(segment
 		(start 101.9875 63.8)
+		(end 117.47 63.8)
+		(width 0.2)
+		(layer "F.Cu")
+		(net 7)
+	)
+	(segment
+		(start 117.47 63.8)
 		(end 120.5875 63.8)
 		(width 0.2)
@@
 	)
 	(segment
-		(start 98.5 63.8)
-		(end 98.5 63.85)
+		(start 135.6 63.8)
+		(end 135.25 63.8)
 		(width 0.2)
 		(layer "F.Cu")
@@
 	)
 	(segment
-		(start 137.4875 65.5)
+		(start 139.1875 63.8)
+		(end 154.3 63.8)
+		(width 0.2)
+		(layer "F.Cu")
+		(net 7)
+	)
+	(segment
+		(start 135.25 63.8)
 		(end 139.1875 63.8)
 		(width 0.2)
@@
 	)
 	(segment
-		(start 139.1875 63.8)
-		(end 157.6 63.8)
+		(start 118.8 65.13)
+		(end 117.47 63.8)
 		(width 0.2)
 		(layer "F.Cu")
@@
 	)
 	(segment
-		(start 157.6 63.8)
-		(end 155.9 65.5)
+		(start 98.5 63.85)
+		(end 98.5 63.8)
 		(width 0.2)
 		(layer "F.Cu")
@@
 	)
 	(segment
-		(start 100.2875 65.5)
-		(end 101.9875 63.8)
+		(start 118.8 65.5)
+		(end 118.8 65.13)
 		(width 0.2)
 		(layer "F.Cu")
