File: _autosave-macroKeyPad.kicad_pcb (KiCad board)
At the start: 2 copper layers, 102.3 x 39.6 mm, 18 parts, among them U1 kb2040

Commit message: wiring
Parts:
- removed G***: LOGO, LOGO
Routing:
- net Row1: track 0.00 -> 66.3 mm, vias 0 -> 4
- net Row0: track 0.00 -> 66.1 mm, vias 0 -> 4
- net Col0: track 0.00 -> 19.5 mm
- net Col2: track 0.00 -> 19.3 mm
- net Col1: track 0.00 -> 19.3 mm
- net Col3: track 0.00 -> 19.3 mm
- net Net-(D6-A): track 0.00 -> 10.1 mm
- net Net-(D5-A): track 0.00 -> 10.1 mm
- net Net-(D7-A): track 0.00 -> 10.1 mm
- net Net-(D8-A): track 0.00 -> 10.1 mm
- net Net-(D4-A): track 0.00 -> 10.0 mm
- net Net-(D3-A): track 0.00 -> 9.99 mm
- net Net-(D2-A): track 0.00 -> 9.99 mm
- net Net-(D1-A): track 0.00 -> 9.99 mm
